File: Hardware/Support-Board-for-TS3008/Support-Board-for-TS3008.kicad_sch (KiCad schematic)
At the start: 53 parts, among them Q1 2N3904S-RTK/PS, SW2 TS-1088R-02026, SW3 TS-1088R-02026, U1 TS64215

Commit message: added libs and finished v1 of PCB
Parts:
- removed H1: (no value), symbol Mechanical:MountingHole_Pad
- removed H2, H3, H4: MountingHole_Pad, symbol Mechanical:MountingHole_Pad
- removed Q1: 2N3904S-RTK/PS, symbol Device:Q_NPN_BCE
- added Q1: (no value), symbol 2N3904S:2N3904S
- C4: value 100NF -> (none)
- C6: value 1UF -> (none)
- SW2, SW3: footprint Copy -> (none)
- U1: footprint BluetoothAudioModule(2)_TS64215 -> (none)
Connections:
- net GNDD: now also Q1.1 (E)
- net MFB: now also Q1.3 (C)
- net at R1.2, R2.2: now also Q1.2 (B)
